File: PCB/SCB.kicad_pcb (KiCad board)
At the start: 2 copper layers, 150 x 195 mm, 48 parts, among them J1 Conn_01x05, J13 Conn_01x04, J14 Conn_01x04, J15 Conn_01x03, J2 Conn_01x05, J3 Conn_01x07, J4 Conn_01x05, J5 Conn_01x07, J6 Conn_01x05, U13 SN74HCT245DWR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

Commit message: Fixed holes in the PCBs
Parts:
- removed the REF** at (29.7, 167.2)
- added REF**: MountingHole_5mm, MountingHole:MountingHole_5mm, F.Cu at (-164.5, -52.0)
- added REF**: MountingHole_5mm, MountingHole:MountingHole_5mm, F.Cu at (-194.5, 36.8)
- added REF**: MountingHole_5mm, MountingHole:MountingHole_5mm, F.Cu at (-124.5, -52.0)
- added REF**: MountingHole_5mm, MountingHole:MountingHole_5mm, F.Cu at (-124.5, -92.0)
- added REF**: MountingHole_5mm, MountingHole:MountingHole_5mm, F.Cu at (-164.5, -92.0)
- moved REF** 259.4 mm to (-94.1, 54.2)
- moved REF** 259.4 mm to (-172.1, 54.2)
- moved REF** 259.4 mm to (-194.5, 54.2)
- moved REF** 259.4 mm to (-94.1, 36.8)
- moved C1 259.1 mm to (-167.0, 23.5)
- moved C2 259.1 mm to (-164.5, -5.00)
- moved C3 259.1 mm to (-161.0, 52.0)
- moved C4 259.1 mm to (-106.5, 52.5)
- moved C5 259.1 mm to (-85.5, 46.5)
- moved C6 259.1 mm to (-124.0, 43.5)
- moved J1 259.1 mm to (-202.6, -46.9)
- moved J13 259.1 mm to (-155.8, 58.4)
- moved J14 259.1 mm to (-109.2, 46.0)
- moved J15 259.1 mm to (-122.0, 30.5)
- moved J5 259.1 mm to (-113.6, 59.8)
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