File: PCB/SCB_normal.kicad_pcb (KiCad board)
At the start: 2 copper layers, 160 x 160 mm, 22 parts, among them J10 Conn_01x05, J11 Conn_01x05, J12 Conn_01x05, J7 Conn_01x05, J8 Conn_01x05, J9 Conn_01x05

Commit message: Fixed holes in the PCBs
Parts:
- added REF**: MountingHole_5mm, MountingHole:MountingHole_5mm, F.Cu at (-255.5, 15.0)
- added REF**: MountingHole_5mm, MountingHole:MountingHole_5mm, F.Cu at (-215.5, 55.0)
- added REF**: MountingHole_5mm, MountingHole:MountingHole_5mm, F.Cu at (-255.5, -25.0)
- added REF**: MountingHole_5mm, MountingHole:MountingHole_5mm, F.Cu at (-215.5, -25.0)
- added REF**: MountingHole_5mm, MountingHole:MountingHole_5mm, F.Cu at (-255.5, 55.0)
- added REF**: MountingHole_5mm, MountingHole:MountingHole_5mm, F.Cu at (-295.5, 55.0)
- added REF**: MountingHole_5mm, MountingHole:MountingHole_5mm, F.Cu at (-215.5, 15.0)
- added REF**: MountingHole_5mm, MountingHole:MountingHole_5mm, F.Cu at (-295.5, 15.0)
- added REF**: MountingHole_5mm, MountingHole:MountingHole_5mm, F.Cu at (-295.5, -25.0)
- moved J12 381.8 mm to (-177.4, 60.1)
- moved J10 381.8 mm to (-260.6, 93.1)
- moved J11 381.8 mm to (-260.6, -63.1)
- moved J7 381.8 mm to (-177.4, 20.1)
- moved J8 381.8 mm to (-333.6, 20.1)
- moved J9 381.8 mm to (-220.6, 93.1)
- moved U21 381.8 mm to (-315.5, -45.0)
- moved U22 381.8 mm to (-315.5, -5.00)
- moved U23 381.8 mm to (-315.5, 35.0)
- moved U24 381.8 mm to (-315.5, 75.0)
- moved U25 381.8 mm to (-275.5, -45.0)
- moved U26 381.8 mm to (-275.5, -5.00)
- moved U27 381.8 mm to (-275.5, 35.0)
- moved U28 381.8 mm to (-275.5, 75.0)
- moved U29 381.8 mm to (-235.5, -45.0)
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Routing:
- net /Matrice 4x4/CC_IN: track 256.2 -> 257.4 mm
- net /Matrice 4x4/L3_IN: track 282.1 -> 283.1 mm
- net /Matrice 4x4/L4_IN: track 398.1 -> 398.9 mm
- net /Matrice 4x4/CB_IN: track 275.2 -> 275.8 mm
